Commit message: Added Sensor

File: models/transportation/transportation.xacro (robot description, xacro)
@@ -1,12 +1,17 @@
 <?xml version='1.0'?>
 <robot name="transportation" xmlns:xacro="http://www.ros.org/wiki/xacro">
-  <xacro:include filename="$(find lunabotics2020)/models/transportation.gazebo" />
-  <xacro:include filename="$(find lunabotics2020)/models/materials.xacro" />
-  <xacro:include filename="$(find lunabotics2020)/models/macros.xacro" />
+<!--http://gazebosim.org/tutorials?tut=guided_i1 for lidar-->
+<!--http://gazebosim.org/tutorials?tut=ros_gzplugins for sensors-->
+  <xacro:include filename="$(find lunabotics2020)/models/transportation/transportation.gazebo" />
+  <xacro:include filename="$(find lunabotics2020)/models/transportation/materials.xacro" />
+  <xacro:include filename="$(find lunabotics2020)/models/transportation/macros.xacro" />
+  <!--Macros-->
+  <xacro:property name="wheel_height" value="-0.05"/>
+  <!--End Macros-->
   <link name='chassis'>
     <pose>0 0 0.1 0 0 0</pose>
     <inertial>
       <mass value="10.0"/>
-      <origin xyz="0.0 0 0.1" rpy=" 0 0 0"/>
+      <origin xyz="0.0 0.0 0.1" rpy="0.0 0.0 0.0"/>
       <inertia
           ixx="0.5" ixy="0" ixz="0"
@@ -17,15 +22,15 @@
     <collision name='collision'>
       <geometry>
-        <box size=".4 .2 .1"/>
+        <box size=".4 .2 .15"/>
       </geometry>
     </collision>
     <visual name='chassis_visual'>
-      <origin xyz="0 0 0" rpy=" 0 0 0"/>
-      <geometry>
-        <box size=".4 .2 .1"/>
-      </geometry>
-    </visual>
-  </link>
-  <link name='front'>
+      <origin xyz="0 0 0" rpy="0 0 0"/>
+      <geometry>
+        <box size=".4 .2 .15"/>
+      </geometry>
+    </visual>
+  </link>
+  <!--link name='front'>
     <collision name='collision'>
       <origin xyz="0 0 0" rpy="0 0 0"/>
@@ -49,7 +54,6 @@
       />
     </inertial>
-  </link>
+  </link-->
   <link name="left_wheel">
-    <!--origin xyz="0.1 0.13 0.1" rpy="0 1.5707 1.5707"/-->
     <collision name="collision">
       <origin xyz="0 0 0" rpy="0 1.5707 1.5707"/>
@@ -75,5 +79,4 @@
   </link>
     <link name="left_rear_wheel">
-    <!--origin xyz="0.1 0.13 0.1" rpy="0 1.5707 1.5707"/-->
     <collision name="collision">
       <origin xyz="0 0 0" rpy="0 1.5707 1.5707"/>
@@ -99,5 +102,4 @@
   </link>
   <link name="right_wheel">
-    <!--origin xyz="0.1 -0.13 0.1" rpy="0 1.5707 1.5707"/-->
     <collision name="collision">
       <origin xyz="0 0 0" rpy="0 1.5707 1.5707"/>
@@ -123,5 +125,4 @@
   </link>
     <link name="right_rear_wheel">
-    <!--origin xyz="0.1 -0.13 0.1" rpy="0 1.5707 1.5707"/-->
     <collision name="collision">
       <origin xyz="0 0 0" rpy="0 1.5707 1.5707"/>
@@ -147,5 +148,5 @@
   </link>
   <joint type="continuous" name="left_wheel_hinge">
-    <origin xyz="0.11 0.15 0" rpy="0 0 0"/>
+    <origin  xyz="0.11 0.15 ${wheel_height}" rpy="0 0 0"/>
     <child link="left_wheel"/>
     <parent link="chassis"/>
@@ -155,5 +156,5 @@
   </joint>
   <joint type="continuous" name="left_rear_wheel_hinge">
-    <origin xyz="-0.11 0.15 0" rpy="0 0 0"/>
+    <origin xyz="-0.11 0.15 ${wheel_height}" rpy="0 0 0"/>
     <child link="left_rear_wheel"/>
     <parent link="chassis"/>
@@ -163,5 +164,5 @@
   </joint>
   <joint type="continuous" name="right_wheel_hinge">
-    <origin xyz="0.11 -0.15 0" rpy="0 0 0"/>
+    <origin xyz="0.11 -0.15 ${wheel_height}" rpy="0 0 0"/>
     <child link="right_wheel"/>
     <parent link="chassis"/>
@@ -171,5 +172,5 @@
   </joint>
   <joint type="continuous" name="right_rear_wheel_hinge">
-    <origin xyz="-0.11 -0.15 0" rpy="0 0 0"/>
+    <origin xyz="-0.11 -0.15 ${wheel_height}" rpy="0 0 0"/>
     <child link="right_rear_wheel"/>
     <parent link="chassis"/>
@@ -178,8 +179,68 @@
     <joint_properties damping="0.0" friction="0.0"/>
   </joint>
-  <joint type="fixed" name="front_fixed">
+  <!--joint type="fixed" name="front_fixed">
     <origin xyz="0.1 0 0.05" rpy="0 0 0"/>
     <child link="front"/>
     <parent link="chassis"/>
+  </joint-->
+  <!--Lidar-->
+  <link name="lidar_base">
+    <collision name="collision">
+      <origin xyz="0 0 0" rpy="0 0 0"/>
+      <geometry>
+        <cylinder radius="0.02" length="0.02"/>
+      </geometry>
+    </collision>
+    <visual name="lidar_base_visual">
+      <origin xyz="0 0 0" rpy="0 0 0"/>
+      <geometry>
+        <cylinder radius="0.02" length="0.02"/>
+      </geometry>
+    </visual>
+    <inertial>
+      <origin xyz="0 0 0" rpy="0 0 0"/>
+      <mass value="0.1"/>
+      <cylinder_inertia m="0.5" r="0.1" h="0.05"/>
+      <inertia
+        ixx="1.0" ixy="0.0" ixz="0.0"
+        iyy="1.0" iyz="0.0"
+        izz="1.0"/>
+    </inertial>
+  </link>
+  <link name="lidar_head">
+    <collision name="collision">
+      <origin xyz="0 0 0" rpy="0 0 0"/>
+      <geometry>
+        <cylinder radius="0.02" length="0.02"/>
+      </geometry>
+    </collision>
+    <visual name="lidar_head_visual">
+      <origin xyz="0 0 0" rpy="0 0 0"/>
+      <geometry>
+        <cylinder radius="0.02" length="0.02"/>
+      </geometry>
+    </visual>
+    <inertial>
+      <origin xyz="0 0 0" rpy="0 0 0"/>
+      <mass value="0.01"/>
+      <cylinder_inertia m="0.5" r="0.1" h="0.05"/>
+      <inertia
+        ixx="0.001" ixy="0.0" ixz="0.0"
+        iyy="0.001" iyz="0.0"
+        izz="0.001"/>
+    </inertial>
+  </link>
+  <joint type="fixed" name="lidar_base_fixed">
+    <origin xyz="0.18 0 0.05" rpy="0 0 0"/>
+    <child link="lidar_base"/>
+    <parent link="chassis"/>
+  </joint>
+  <joint type="continuous" name="lidar_head_continuous">
+    <origin xyz="0 0 0.02" rpy="0 0 0"/>
+    <child link="lidar_head"/>
+    <parent link="lidar_base"/>
+    <axis xyz="0 0 1" rpy="0 0 0"/>
+    <limit effort="100000000000" velocity="100"/>
+    <joint_properties damping="0.0" friction="0.0"/>
   </joint>
 </robot>

Commit message: Put field model directly into world file

File: models/transportation/transportation.xacro (robot description, xacro)
@@ -8,4 +8,5 @@
   <!--Macros-->
   <xacro:property name="wheel_height" value="-0.05"/>
+  <xacro:property name="lidar_base_size" value="0.05 0.05 0.025"/>
   <!--End Macros-->
   <link name='chassis'>
@@ -32,20 +33,134 @@
     </visual>
   </link>
-  <!--link name='front'>
-    <collision name='collision'>
-      <origin xyz="0 0 0" rpy="0 0 0"/>
-      <geometry>
-        <box size='.1 .1 0.02'/>
-      </geometry>
-    </collision>
-    <visual name='front_visual'>
-      <origin xyz="0 0 0" rpy="0 0 0"/>
-      <geometry>
-        <box size="0.1 0.1 0.02"/>
-      </geometry>
-    </visual>
-    <inertial>
-      <mass value="10.0"/>
-      <origin xyz="0.0 0 0" rpy=" 0 0 0"/>
+  <link name="left_wheel">
+    <collision name="collision">
+      <origin xyz="0 0 0" rpy="0 1.5707 1.5707"/>
+      <geometry>
+        <cylinder radius="0.1" length="0.05"/>
+      </geometry>
+    </collision>
+    <visual name="left_wheel_visual">
+      <origin xyz="0 0 0" rpy="0 1.5707 1.5707"/>
+      <geometry>
+        <cylinder radius="0.1" length="0.05"/>
+      </geometry>
+    </visual>
+    <inertial>
+      <origin xyz="0 0 0" rpy="0 1.5707 1.5707"/>
+      <mass value="5"/>
+      <cylinder_inertia m="5" r="0.1" h="0.05"/>
+      <inertia
+        ixx="1.0" ixy="0.0" ixz="0.0"
+        iyy="1.0" iyz="0.0"
+        izz="1.0"/>
+    </inertial>
+  </link>
+    <link name="left_rear_wheel">
+    <collision name="collision">
+      <origin xyz="0 0 0" rpy="0 1.5707 1.5707"/>
+      <geometry>
+        <cylinder radius="0.1" length="0.05"/>
+      </geometry>
+    </collision>
+    <visual name="left_rear_wheel_visual">
+      <origin xyz="0 0 0" rpy="0 1.5707 1.5707"/>
+      <geometry>
+        <cylinder radius="0.1" length="0.05"/>
+      </geometry>
+    </visual>
+    <inertial>
+      <origin xyz="0 0 0" rpy="0 1.5707 1.5707"/>
+      <mass value="5"/>
+      <cylinder_inertia m="5" r="0.1" h="0.05"/>
+      <inertia
+        ixx="1.0" ixy="0.0" ixz="0.0"
+        iyy="1.0" iyz="0.0"
+        izz="1.0"/>
+    </inertial>
+  </link>
+  <link name="right_wheel">
+    <collision name="collision">
+      <origin xyz="0 0 0" rpy="0 1.5707 1.5707"/>
+      <geometry>
+        <cylinder radius="0.1" length="0.05"/>
+      </geometry>
+    </collision>
+    <visual name="right_wheel_visual">
+      <origin xyz="0 0 0" rpy="0 1.5707 1.5707"/>
+      <geometry>
+        <cylinder radius="0.1" length="0.05"/>
+      </geometry>
+    </visual>
+    <inertial>
+      <origin xyz="0 0 0" rpy="0 1.5707 1.5707"/>
+      <mass value="5"/>
+      <cylinder_inertia m="5" r="0.1" h="0.05"/>
+      <inertia
+        ixx="1.0" ixy="0.0" ixz="0.0"
+        iyy="1.0" iyz="0.0"
+        izz="1.0"/>
+    </inertial>
+  </link>
+    <link name="right_rear_wheel">
+    <collision name="collision">
+      <origin xyz="0 0 0" rpy="0 1.5707 1.5707"/>
+      <geometry>
+        <cylinder radius="0.1" length="0.05"/>
+      </geometry>
+    </collision>
+    <visual name="right_rear_wheel_visual">
+      <origin xyz="0 0 0" rpy="0 1.5707 1.5707"/>
+      <geometry>
+        <cylinder radius="0.1" length="0.05"/>
+      </geometry>
+    </visual>
+    <inertial>
+      <origin xyz="0 0 0" rpy="0 1.5707 1.5707"/>
+      <mass value="5"/>
+      <cylinder_inertia m="5" r="0.1" h="0.05"/>
+      <inertia
+        ixx="1.0" ixy="0.0" ixz="0.0"
+        iyy="1.0" iyz="0.0"
+        izz="1.0"/>
+    </inertial>
+  </link>
+  <joint type="continuous" name="left_wheel_hinge">
+    <origin  xyz="0.11 0.15 ${wheel_height}" rpy="0 0 0"/>
+    <child link="left_wheel"/>
+    <parent link="chassis"/>
+    <axis xyz="0 1 0" rpy="0 0 0"/>
+    <limit effort="100" velocity="100"/>
+    <joint_properties damping="0.0" friction="0.0"/>
+  </joint>
+  <joint type="continuous" name="left_rear_wheel_hinge">
+    <origin xyz="-0.11 0.15 ${wheel_height}" rpy="0 0 0"/>
+    <child link="left_rear_wheel"/>
+    <parent link="chassis"/>
+    <axis xyz="0 1 0" rpy="0 0 0"/>
+    <limit effort="100" velocity="100"/>
+    <joint_properties damping="0.0" friction="0.0"/>
+  </joint>
+  <joint type="continuous" name="right_wheel_hinge">
+    <origin xyz="0.11 -0.15 ${wheel_height}" rpy="0 0 0"/>
+    <child link="right_wheel"/>
+    <parent link="chassis"/>
+    <axis xyz="0 1 0" rpy="0 0 0"/>
+    <limit effort="100" velocity="100"/>
+    <joint_properties damping="0.0" friction="0.0"/>
+  </joint>
+  <joint type="continuous" name="right_rear_wheel_hinge">
+    <origin xyz="-0.11 -0.15 ${wheel_height}" rpy="0 0 0"/>
+    <child link="right_rear_wheel"/>
+    <parent link="chassis"/>
+    <axis xyz="0 1 0" rpy="0 0 0"/>
+    <limit effort="100" velocity="100"/>
+    <joint_properties damping="0.0" friction="0.0"/>
+  </joint>
+  <!--====  Lidar  ========================================-->
+  <link name='lidar_base'>
+    <pose>0 0 0.1 0 0 0</pose>
+    <inertial>
+      <mass value="1.0"/>
+      <origin xyz="0.0 0.0 0.1" rpy="0.0 0.0 0.0"/>
       <inertia
           ixx="0.5" ixy="0" ixz="0"
@@ -54,136 +169,17 @@
       />
     </inertial>
-  </link-->
-  <link name="left_wheel">
-    <collision name="collision">
-      <origin xyz="0 0 0" rpy="0 1.5707 1.5707"/>
-      <geometry>
-        <cylinder radius="0.1" length="0.05"/>
-      </geometry>
-    </collision>
-    <visual name="left_wheel_visual">
-      <origin xyz="0 0 0" rpy="0 1.5707 1.5707"/>
-      <geometry>
-        <cylinder radius="0.1" length="0.05"/>
-      </geometry>
-    </visual>
-    <inertial>
-      <origin xyz="0 0 0" rpy="0 1.5707 1.5707"/>
-      <mass value="5"/>
-      <cylinder_inertia m="5" r="0.1" h="0.05"/>
-      <inertia
-        ixx="1.0" ixy="0.0" ixz="0.0"
-        iyy="1.0" iyz="0.0"
-        izz="1.0"/>
-    </inertial>
-  </link>
-    <link name="left_rear_wheel">
-    <collision name="collision">
-      <origin xyz="0 0 0" rpy="0 1.5707 1.5707"/>
-      <geometry>
-        <cylinder radius="0.1" length="0.05"/>
-      </geometry>
-    </collision>
-    <visual name="left_rear_wheel_visual">
-      <origin xyz="0 0 0" rpy="0 1.5707 1.5707"/>
-      <geometry>
-        <cylinder radius="0.1" length="0.05"/>
-      </geometry>
-    </visual>
-    <inertial>
-      <origin xyz="0 0 0" rpy="0 1.5707 1.5707"/>
-      <mass value="5"/>
-      <cylinder_inertia m="5" r="0.1" h="0.05"/>
-      <inertia
-        ixx="1.0" ixy="0.0" ixz="0.0"
-        iyy="1.0" iyz="0.0"
-        izz="1.0"/>
-    </inertial>
-  </link>
-  <link name="right_wheel">
-    <collision name="collision">
-      <origin xyz="0 0 0" rpy="0 1.5707 1.5707"/>
-      <geometry>
-        <cylinder radius="0.1" length="0.05"/>
-      </geometry>
-    </collision>
-    <visual name="right_wheel_visual">
-      <origin xyz="0 0 0" rpy="0 1.5707 1.5707"/>
-      <geometry>
-        <cylinder radius="0.1" length="0.05"/>
-      </geometry>
-    </visual>
-    <inertial>
-      <origin xyz="0 0 0" rpy="0 1.5707 1.5707"/>
-      <mass value="5"/>
-      <cylinder_inertia m="5" r="0.1" h="0.05"/>
-      <inertia
-        ixx="1.0" ixy="0.0" ixz="0.0"
-        iyy="1.0" iyz="0.0"
-        izz="1.0"/>
-    </inertial>
-  </link>
-    <link name="right_rear_wheel">
-    <collision name="collision">
-      <origin xyz="0 0 0" rpy="0 1.5707 1.5707"/>
-      <geometry>
-        <cylinder radius="0.1" length="0.05"/>
-      </geometry>
-    </collision>
-    <visual name="right_rear_wheel_visual">
-      <origin xyz="0 0 0" rpy="0 1.5707 1.5707"/>
-      <geometry>
-        <cylinder radius="0.1" length="0.05"/>
-      </geometry>
-    </visual>
-    <inertial>
-      <origin xyz="0 0 0" rpy="0 1.5707 1.5707"/>
-      <mass value="5"/>
-      <cylinder_inertia m="5" r="0.1" h="0.05"/>
-      <inertia
-        ixx="1.0" ixy="0.0" ixz="0.0"
-        iyy="1.0" iyz="0.0"
-        izz="1.0"/>
-    </inertial>
-  </link>
-  <joint type="continuous" name="left_wheel_hinge">
-    <origin  xyz="0.11 0.15 ${wheel_height}" rpy="0 0 0"/>
-    <child link="left_wheel"/>
-    <parent link="chassis"/>
-    <axis xyz="0 1 0" rpy="0 0 0"/>
-    <limit effort="100" velocity="100"/>
-    <joint_properties damping="0.0" friction="0.0"/>
-  </joint>
-  <joint type="continuous" name="left_rear_wheel_hinge">
-    <origin xyz="-0.11 0.15 ${wheel_height}" rpy="0 0 0"/>
-    <child link="left_rear_wheel"/>
-    <parent link="chassis"/>
-    <axis xyz="0 1 0" rpy="0 0 0"/>
-    <limit effort="100" velocity="100"/>
-    <joint_properties damping="0.0" friction="0.0"/>
-  </joint>
-  <joint type="continuous" name="right_wheel_hinge">
-    <origin xyz="0.11 -0.15 ${wheel_height}" rpy="0 0 0"/>
-    <child link="right_wheel"/>
-    <parent link="chassis"/>
-    <axis xyz="0 1 0" rpy="0 0 0"/>
-    <limit effort="100" velocity="100"/>
-    <joint_properties damping="0.0" friction="0.0"/>
-  </joint>
-  <joint type="continuous" name="right_rear_wheel_hinge">
-    <origin xyz="-0.11 -0.15 ${wheel_height}" rpy="0 0 0"/>
-    <child link="right_rear_wheel"/>
-    <parent link="chassis"/>
-    <axis xyz="0 1 0" rpy="0 0 0"/>
-    <limit effort="100" velocity="100"/>
-    <joint_properties damping="0.0" friction="0.0"/>
-  </joint>
-  <!--joint type="fixed" name="front_fixed">
-    <origin xyz="0.1 0 0.05" rpy="0 0 0"/>
-    <child link="front"/>
-    <parent link="chassis"/>
-  </joint-->
-  <!--Lidar-->
-  <link name="lidar_base">
+    <collision name='collision'>
+      <geometry>
+        <box size="${lidar_base_size}"/>
+      </geometry>
+    </collision>
+    <visual name='lidar_base_pivot_visual'>
+      <origin xyz="0 0 0" rpy="0 0 0"/>
+      <geometry>
+        <box size="${lidar_base_size}"/>
+      </geometry>
+    </visual>
+  </link>
+  <link name="lidar">
     <collision name="collision">
       <origin xyz="0 0 0" rpy="0 0 0"/>
@@ -192,28 +188,5 @@
       </geometry>
     </collision>
-    <visual name="lidar_base_visual">
-      <origin xyz="0 0 0" rpy="0 0 0"/>
-      <geometry>
-        <cylinder radius="0.02" length="0.02"/>
-      </geometry>
-    </visual>
-    <inertial>
-      <origin xyz="0 0 0" rpy="0 0 0"/>
-      <mass value="0.1"/>
-      <cylinder_inertia m="0.5" r="0.1" h="0.05"/>
-      <inertia
-        ixx="1.0" ixy="0.0" ixz="0.0"
-        iyy="1.0" iyz="0.0"
-        izz="1.0"/>
-    </inertial>
-  </link>
-  <link name="lidar_head">
-    <collision name="collision">
-      <origin xyz="0 0 0" rpy="0 0 0"/>
-      <geometry>
-        <cylinder radius="0.02" length="0.02"/>
-      </geometry>
-    </collision>
-    <visual name="lidar_head_visual">
+    <visual name="lidar_visual">
       <origin xyz="0 0 0" rpy="0 0 0"/>
       <geometry>
@@ -226,21 +199,18 @@
       <cylinder_inertia m="0.5" r="0.1" h="0.05"/>
       <inertia
-        ixx="0.001" ixy="0.0" ixz="0.0"
-        iyy="0.001" iyz="0.0"
-        izz="0.001"/>
+        ixx="1.0" ixy="0.0" ixz="0.0"
+        iyy="1.0" iyz="0.0"
+        izz="1.0"/>
     </inertial>
   </link>
   <joint type="fixed" name="lidar_base_fixed">
-    <origin xyz="0.18 0 0.05" rpy="0 0 0"/>
+    <origin xyz="0.18 0 0.0895" rpy="0 0 0"/>
     <child link="lidar_base"/>
     <parent link="chassis"/>
   </joint>
-  <joint type="continuous" name="lidar_head_continuous">
-    <origin xyz="0 0 0.02" rpy="0 0 0"/>
-    <child link="lidar_head"/>
+  <joint type="fixed" name="lidar_fixed">
+    <origin xyz="0 0 0.0128" rpy="0 0 0"/>
+    <child link="lidar"/>
     <parent link="lidar_base"/>
-    <axis xyz="0 0 1" rpy="0 0 0"/>
-    <limit effort="100000000000" velocity="100"/>
-    <joint_properties damping="0.0" friction="0.0"/>
   </joint>
 </robot>

Commit message: Four Wheeled Arcade Drive

File: models/transportation/transportation.xacro (robot description, xacro)
@@ -9,14 +9,17 @@
   <xacro:property name="wheel_height" value="-0.05"/>
   <xacro:property name="lidar_base_size" value="0.05 0.05 0.025"/>
+  <xacro:property name="wheel_inertia_ixx" value="0.025"/>
+  <xacro:property name="wheel_inertia_iyy" value="0.025"/>
+  <xacro:property name="wheel_inertia_izz" value="0.025"/>
   <!--End Macros-->
   <link name='chassis'>
     <pose>0 0 0.1 0 0 0</pose>
     <inertial>
-      <mass value="10.0"/>
-      <origin xyz="0.0 0.0 0.1" rpy="0.0 0.0 0.0"/>
-      <inertia
-          ixx="0.5" ixy="0" ixz="0"
-          iyy="1.0" iyz="0"
-          izz="0.1"
+      <mass value="20.0"/>
+      <origin xyz="0.0 0.0 0.0" rpy="0.0 0.0 0.0"/>
+      <inertia
+          ixx="0.4" ixy="0" ixz="0"
+          iyy="0.2" iyz="0"
+          izz="0.15"
       />
     </inertial>
@@ -51,7 +54,7 @@
       <cylinder_inertia m="5" r="0.1" h="0.05"/>
       <inertia
-        ixx="1.0" ixy="0.0" ixz="0.0"
-        iyy="1.0" iyz="0.0"
-        izz="1.0"/>
+        ixx="${wheel_inertia_ixx}" ixy="0.0" ixz="0.0"
+        iyy="${wheel_inertia_iyy}" iyz="0.0"
+        izz="${wheel_inertia_izz}"/>
     </inertial>
   </link>
@@ -74,7 +77,7 @@
       <cylinder_inertia m="5" r="0.1" h="0.05"/>
       <inertia
-        ixx="1.0" ixy="0.0" ixz="0.0"
-        iyy="1.0" iyz="0.0"
-        izz="1.0"/>
+        ixx="${wheel_inertia_ixx}" ixy="0.0" ixz="0.0"
+        iyy="${wheel_inertia_iyy}" iyz="0.0"
+        izz="${wheel_inertia_izz}"/>
     </inertial>
   </link>
@@ -97,7 +100,7 @@
       <cylinder_inertia m="5" r="0.1" h="0.05"/>
       <inertia
-        ixx="1.0" ixy="0.0" ixz="0.0"
-        iyy="1.0" iyz="0.0"
-        izz="1.0"/>
+        ixx="${wheel_inertia_ixx}" ixy="0.0" ixz="0.0"
+        iyy="${wheel_inertia_iyy}" iyz="0.0"
+        izz="${wheel_inertia_izz}"/>
     </inertial>
   </link>
@@ -120,7 +123,7 @@
       <cylinder_inertia m="5" r="0.1" h="0.05"/>
       <inertia
-        ixx="1.0" ixy="0.0" ixz="0.0"
-        iyy="1.0" iyz="0.0"
-        izz="1.0"/>
+        ixx="${wheel_inertia_ixx}" ixy="0.0" ixz="0.0"
+        iyy="${wheel_inertia_iyy}" iyz="0.0"
+        izz="${wheel_inertia_izz}"/>
     </inertial>
   </link>
@@ -161,10 +164,10 @@
     <pose>0 0 0.1 0 0 0</pose>
     <inertial>
-      <mass value="1.0"/>
+      <mass value="0.01"/>
       <origin xyz="0.0 0.0 0.1" rpy="0.0 0.0 0.0"/>
       <inertia
-          ixx="0.5" ixy="0" ixz="0"
-          iyy="1.0" iyz="0"
-          izz="0.1"
+          ixx="0.05" ixy="0" ixz="0"
+          iyy="0.05" iyz="0"
+          izz="0.025"
       />
     </inertial>
@@ -199,7 +202,7 @@
       <cylinder_inertia m="0.5" r="0.1" h="0.05"/>
       <inertia
-        ixx="1.0" ixy="0.0" ixz="0.0"
-        iyy="1.0" iyz="0.0"
-        izz="1.0"/>
+        ixx="0.02" ixy="0.0" ixz="0.0"
+        iyy="0.02" iyz="0.0"
+        izz="0.02"/>
     </inertial>
   </link>
