Commit message: Fixed Model

File: description/dug.xacro (robot description, xacro)
@@ -8,5 +8,5 @@
   <!--End Macros-->
   <link name='chassis'>
-    <pose>0 0 0.1 0 0 0</pose>
+    <!--pose>0 0 0.1 0 0 0</pose-->
     <inertial>
       <mass value="20.0"/>
@@ -124,5 +124,5 @@
   <joint type="continuous" name="left_front_wheel_hinge">
     <origin  xyz="0.11 0.15 ${wheel_height}" rpy="0 0 0"/>
-    <child link="left_wheel"/>
+    <child link="left_front_wheel"/>
     <parent link="chassis"/>
     <axis xyz="0 1 0" rpy="0 0 0"/>
@@ -140,5 +140,5 @@
   <joint type="continuous" name="right_front_wheel_hinge">
     <origin xyz="0.11 -0.15 ${wheel_height}" rpy="0 0 0"/>
-    <child link="right_wheel"/>
+    <child link="right_front_wheel"/>
     <parent link="chassis"/>
     <axis xyz="0 1 0" rpy="0 0 0"/>

File: description/test.xacro (robot description, xacro)
@@ -2,4 +2,13 @@
 <robot name="test" xmlns:xacro="http://www.ros.org/wiki/xacro">
   <link name='chassis'>
+  <inertial>
+      <mass value="20.0"/>
+      <origin xyz="0.0 0.0 0.0" rpy="0.0 0.0 0.0"/>
+      <inertia
+          ixx="0.4" ixy="0" ixz="0"
+          iyy="0.2" iyz="0"
+          izz="0.15"
+      />
+    </inertial>
     <collision name='collision'>
       <geometry>

Commit message: Working on diff_drive in gazebo

File: description/dug.xacro (robot description, xacro)
@@ -122,5 +122,5 @@
     </inertial>
   </link>
-  <joint type="continuous" name="left_front_wheel_hinge">
+  <joint type="continuous" name="left_front_wheel_joint">
     <origin  xyz="0.11 0.15 ${wheel_height}" rpy="0 0 0"/>
     <child link="left_front_wheel"/>
@@ -130,5 +130,14 @@
     <joint_properties damping="0.0" friction="0.0"/>
   </joint>
-  <joint type="continuous" name="left_rear_wheel_hinge">
+  <transmission name="left_front_wheel_transm">
+    <type>transmission_interface/SimpleTransmission</type>
+    <joint name="left_front_wheel_joint">
+      <hardwareInterface>hardware_interface/VelocityJointInterface</hardwareInterface>
+    </joint>
+    <actuator name="left_front_wheel_motor">
+      <hardwareInterface>hardware_interface/VelocityJointInterface</hardwareInterface>
+   </actuator>
+  </transmission>
+  <joint type="continuous" name="left_rear_wheel_joint">
     <origin xyz="-0.11 0.15 ${wheel_height}" rpy="0 0 0"/>
     <child link="left_rear_wheel"/>
@@ -138,5 +147,14 @@
     <joint_properties damping="0.0" friction="0.0"/>
   </joint>
-  <joint type="continuous" name="right_front_wheel_hinge">
+  <transmission name="left_rear_wheel_transm">
+    <type>transmission_interface/SimpleTransmission</type>
+    <joint name="left_rear_wheel_joint">
+      <hardwareInterface>hardware_interface/VelocityJointInterface</hardwareInterface>
+    </joint>
+    <actuator name="left_rear_wheel_motor">
+      <hardwareInterface>hardware_interface/VelocityJointInterface</hardwareInterface>
+   </actuator>
+  </transmission>
+  <joint type="continuous" name="right_front_wheel_joint">
     <origin xyz="0.11 -0.15 ${wheel_height}" rpy="0 0 0"/>
     <child link="right_front_wheel"/>
@@ -146,5 +164,14 @@
     <joint_properties damping="0.0" friction="0.0"/>
   </joint>
-  <joint type="continuous" name="right_rear_wheel_hinge">
+  <transmission name="right_front_wheel_transm">
+    <type>transmission_interface/SimpleTransmission</type>
+    <joint name="right_front_wheel_joint">
+      <hardwareInterface>hardware_interface/VelocityJointInterface</hardwareInterface>
+    </joint>
+    <actuator name="right_front_wheel_motor">
+      <hardwareInterface>hardware_interface/VelocityJointInterface</hardwareInterface>
+   </actuator>
+  </transmission>
+  <joint type="continuous" name="right_rear_wheel_joint">
     <origin xyz="-0.11 -0.15 ${wheel_height}" rpy="0 0 0"/>
     <child link="right_rear_wheel"/>
@@ -154,3 +181,12 @@
     <joint_properties damping="0.0" friction="0.0"/>
   </joint>
+  <transmission name="right_rear_wheel_transm">
+    <type>transmission_interface/SimpleTransmission</type>
+    <joint name="right_rear_wheel_joint">
+      <hardwareInterface>hardware_interface/VelocityJointInterface</hardwareInterface>
+    </joint>
+    <actuator name="right_rear_wheel_motor">
+      <hardwareInterface>hardware_interface/VelocityJointInterface</hardwareInterface>
+   </actuator>
+  </transmission>
 </robot>

File: description/test.xacro (robot description, xacro)
@@ -24,2 +24,7 @@
   </link>
 </robot>
+<gazebo>
+  <plugin name="gazebo_ros_control" filename="libgazebo_ros_control.so">
+    <robotNamespace>/dug</robotNamespace>
+  </plugin>
+</gazebo>

Commit message: began work on Hardware Interface

File: description/dug.xacro (robot description, xacro)
@@ -7,6 +7,6 @@
   <xacro:property name="wheel_inertia_izz" value="0.025"/>
   <!--End Macros-->
+  <!--VISUAL AND INERTIAL-->
   <link name='chassis'>
-    <!--pose>0 0 0.1 0 0 0</pose-->
     <inertial>
       <mass value="20.0"/>
@@ -53,5 +53,5 @@
     </inertial>
   </link>
-    <link name="left_rear_wheel">
+  <link name="left_rear_wheel">
     <collision name="collision">
       <origin xyz="0 0 0" rpy="0 1.5707 1.5707"/>
@@ -99,5 +99,5 @@
     </inertial>
   </link>
-    <link name="right_rear_wheel">
+  <link name="right_rear_wheel">
     <collision name="collision">
       <origin xyz="0 0 0" rpy="0 1.5707 1.5707"/>
@@ -122,4 +122,5 @@
     </inertial>
   </link>
+  <!--JOINTS, TRANSMISSIONS AND GAZEBO PLUGINS-->
   <joint type="continuous" name="left_front_wheel_joint">
     <origin  xyz="0.11 0.15 ${wheel_height}" rpy="0 0 0"/>
@@ -190,4 +191,19 @@
    </actuator>
   </transmission>
+  <gazebo reference="chassis">
+    <material>Gazebo/Blue</material>
+  </gazebo>
+  <gazebo reference="left_front_wheel">
+    <material>Gazebo/Grey</material>
+  </gazebo>
+  <gazebo reference="right_front_wheel">
+    <material>Gazebo/Grey</material>
+  </gazebo>
+  <gazebo reference="left_rear_wheel">
+    <material>Gazebo/Grey</material>
+  </gazebo>
+  <gazebo reference="right_rear_wheel">
+    <material>Gazebo/Grey</material>
+  </gazebo>
   <gazebo>
     <plugin name="gazebo_ros_control" filename="libgazebo_ros_control.so">

Commit message: Added SLRS to simulation

File: description/dug.xacro (robot description, xacro)
@@ -2,8 +2,16 @@
 <robot name="dug" xmlns:xacro="http://www.ros.org/wiki/xacro">
   <!--Macros-->
-  <xacro:property name="wheel_height" value="-0.05"/>
+  <xacro:property name="chassis_height" value="0.1"/>
+  <xacro:property name="chassis_width" value="0.34"/>
+  <xacro:property name="chassis_length" value="0.35"/>
+  <xacro:property name="wheel_height" value="-0.07"/>
+  <xacro:property name="wheel_y" value="0.2"/>
+  <xacro:property name="wheel_x" value="0.11"/>
   <xacro:property name="wheel_inertia_ixx" value="0.025"/>
   <xacro:property name="wheel_inertia_iyy" value="0.025"/>
   <xacro:property name="wheel_inertia_izz" value="0.025"/>
+  <xacro:property name="slrs_one_radius" value="0.02"/>
+  <xacro:property name="slrs_two_radius" value="0.05"/>
+  <xacro:property name="slrs_pole_height" value="0.3"/>
   <!--End Macros-->
   <!--VISUAL AND INERTIAL-->
@@ -20,5 +28,5 @@
     <collision name='collision'>
       <geometry>
-        <box size=".4 .2 .15"/>
+        <box size="${chassis_length} ${chassis_width} ${chassis_height}"/>
       </geometry>
     </collision>
@@ -26,5 +34,5 @@
       <origin xyz="0 0 0" rpy="0 0 0"/>
       <geometry>
-        <box size=".4 .2 .15"/>
+        <box size="${chassis_length} ${chassis_width} ${chassis_height}"/>
       </geometry>
     </visual>
@@ -114,4 +122,51 @@
     <inertial>
       <origin xyz="0 0 0" rpy="0 1.5707 1.5707"/>
+      <mass value="5"/>
+      <cylinder_inertia m="5" r="0.1" h="0.05"/>
+      <inertia
+        ixx="${wheel_inertia_ixx}" ixy="0.0" ixz="0.0"
+        iyy="${wheel_inertia_iyy}" iyz="0.0"
+        izz="${wheel_inertia_izz}"/>
+    </inertial>
+  </link>
+  <!--SLRS POLES-->
+  <link name="slrs_pole_one">
+    <collision name="collision">
+      <origin xyz="0 0 0" rpy="0 0 0"/>
+      <geometry>
+        <cylinder radius="${slrs_one_radius}" length="${slrs_pole_height}"/>
+      </geometry>
+    </collision>
+    <visual name="slrs_one_visual">
+      <origin xyz="0 0 0" rpy="0 0 0"/>
+      <geometry>
+        <cylinder radius="${slrs_one_radius}" length="${slrs_pole_height}"/>
+      </geometry>
+    </visual>
+    <inertial>
+      <origin xyz="0 0 0" rpy="0 0 0"/>
+      <mass value="5"/>
+      <cylinder_inertia m="5" r="0.1" h="0.05"/>
+      <inertia
+        ixx="${wheel_inertia_ixx}" ixy="0.0" ixz="0.0"
+        iyy="${wheel_inertia_iyy}" iyz="0.0"
+        izz="${wheel_inertia_izz}"/>
+    </inertial>
+  </link>
+  <link name="slrs_pole_two">
+    <collision name="collision">
+      <origin xyz="0 0 0" rpy="0 0 0"/>
+      <geometry>
+        <cylinder radius="${slrs_two_radius}" length="${slrs_pole_height}"/>
+      </geometry>
+    </collision>
+    <visual name="slrs_two_visual">
+      <origin xyz="0 0 0" rpy="0 0 0"/>
+      <geometry>
+        <cylinder radius="${slrs_two_radius}" length="${slrs_pole_height}"/>
+      </geometry>
+    </visual>
+    <inertial>
+      <origin xyz="0 0 0" rpy="0 0 0"/>
       <mass value="5"/>
       <cylinder_inertia m="5" r="0.1" h="0.05"/>
@@ -124,5 +179,5 @@
   <!--JOINTS, TRANSMISSIONS AND GAZEBO PLUGINS-->
   <joint type="continuous" name="left_front_wheel_joint">
-    <origin  xyz="0.11 0.15 ${wheel_height}" rpy="0 0 0"/>
+    <origin  xyz="${wheel_x} ${wheel_y} ${wheel_height}" rpy="0 0 0"/>
     <child link="left_front_wheel"/>
     <parent link="chassis"/>
@@ -141,5 +196,5 @@
   </transmission>
   <joint type="continuous" name="left_rear_wheel_joint">
-    <origin xyz="-0.11 0.15 ${wheel_height}" rpy="0 0 0"/>
+    <origin xyz="-${wheel_x} ${wheel_y} ${wheel_height}" rpy="0 0 0"/>
     <child link="left_rear_wheel"/>
     <parent link="chassis"/>
@@ -158,5 +213,5 @@
   </transmission>
   <joint type="continuous" name="right_front_wheel_joint">
-    <origin xyz="0.11 -0.15 ${wheel_height}" rpy="0 0 0"/>
+    <origin xyz="${wheel_x} -${wheel_y} ${wheel_height}" rpy="0 0 0"/>
     <child link="right_front_wheel"/>
     <parent link="chassis"/>
@@ -175,5 +230,5 @@
   </transmission>
   <joint type="continuous" name="right_rear_wheel_joint">
-    <origin xyz="-0.11 -0.15 ${wheel_height}" rpy="0 0 0"/>
+    <origin xyz="-${wheel_x} -${wheel_y} ${wheel_height}" rpy="0 0 0"/>
     <child link="right_rear_wheel"/>
     <parent link="chassis"/>
@@ -191,4 +246,21 @@
    </actuator>
   </transmission>
+  <xacro:property name="chassis_height_half" value="${chassis_height / 2}"/>
+  <joint type="fixed" name="slrs_pole_one_fixed">
+    <origin xyz="-${chassis_length / 2 - slrs_one_radius}
+                ${chassis_width / 2 - slrs_one_radius}
+                ${slrs_pole_height / 2 + chassis_height_half}"
+            rpy="0 0 0"/>
+    <child link="slrs_pole_one"/>
+    <parent link="chassis"/>
+  </joint>
+  <joint type="fixed" name="slrs_pole_two_fixed">
+    <origin xyz="-${chassis_length / 2 - slrs_two_radius}
+                -${chassis_width / 2 - slrs_two_radius}
+                ${slrs_pole_height / 2 + chassis_height_half}"
+            rpy="0 0 0"/>
+    <child link="slrs_pole_two"/>
+    <parent link="chassis"/>
+  </joint>
   <gazebo reference="chassis">
     <material>Gazebo/Blue</material>
